File: A_Key_V1.1.sch (KiCad schematic (older format))
At the start: 149 parts, among them J1 AVR-ISP-6, J2 TYPE-C-31-M12_13, SW1 SW_Push, SW10 [>], SW11 [Win], SW12 [2], SW13 [W], SW14 [S], SW15 [Z], SW16 [Alt], SW17 [3], SW18 [E], SW19 [D], SW2 [\\], SW20 [X], SW21 [4], SW22 [R], SW23 [F], SW24 [C], SW25 [5], SW26 [T], SW27 [G], SW28 [V], SW29 [6], SW3 [LTab], SW30 [Y], SW31 [H], SW32 [B], SW33 [Space], SW34 [7], SW35 [U], SW36 [J], SW37 [N], SW38 [8], SW39 [I], SW4 [LCaps], SW40 [K], SW41 [M], SW42 [9], SW43 [O], SW44 [L], SW45 [;], SW46 [0], SW47 [P], SW48 [Ñ], SW49 [:], SW5 [LShift], SW50 [AltGr], SW51 [?], SW52 [^], SW53 [¨], SW54 [_], SW55 [Win], SW56 [¿], SW57 [*], SW58 [Ç], SW59 [RShift], SW6 [LCtrl], SW60 [Menu], SW61 [Backspc], SW62 [Enter1.5], SW63 [Ctrl2], SW64 [Unass], SW65 [Unass1.25], SW7 [1], SW8 [Q], SW9 [A], U1 ATmega32U4-AU, Y1 Crystal

Commit message: PCB Layout almost finished
Parts:
- removed J2: TYPE-C-31-M12_13, TYPE-C-31-M-12:HRO_TYPE-C-31-M-12, symbol acheronSymbols:TYPE-C-31-M12_13
- removed R6, R7: 5k, Resistor_SMD:R_0805_2012Metric_Pad1.20x1.40mm_HandSolder, symbol Device:R_Small
- removed R8, R9: 22k, Resistor_SMD:R_0805_2012Metric_Pad1.20x1.40mm_HandSolder, symbol Device:R_Small
- added C10: 100n, Capacitor_SMD:C_0805_2012Metric_Pad1.18x1.45mm_HandSolder, symbol Device:C_Small
- added J3: TYPE-C-31-M-12, TYPE-C-31-M-12:HRO_TYPE-C-31-M-12, symbol TYPE-C-31-M-12:TYPE-C-31-M-12
- added R1, R11: 5k, Resistor_SMD:R_0805_2012Metric_Pad1.20x1.40mm_HandSolder, symbol Device:R_Small
- added R10, R2: 22k, Resistor_SMD:R_0805_2012Metric_Pad1.20x1.40mm_HandSolder, symbol Device:R_Small
- C4: value 0.1u -> 10u
- C5: value 0.1u -> 1u
- C7, C8: value 0.1u -> 100n
- C9: value 10u -> 1u
Connections:
- net +5V: now also U1.42 (AREF), C10.1, J3.A4B9 (VBUS), J3.B4A9 (VBUS)
- net Col_13: now also SW65.1 (Col); no longer D13.1 (K), D14.1 (K), D18.1 (K), D19.1 (K), D22.1 (K), D23.1 (K), D26.1 (K), D27.1 (K), D3.1 (K), D30.1 (K), D31.1 (K), D35.1 (K), D36.1 (K), D39.1 (K), D4.1 (K), D40.1 (K), D43.1 (K), D44.1 (K), D47.1 (K), D48.1 (K), D52.1 (K), D53.1 (K), D57.1 (K), D58.1 (K), D63.1 (K), D64.1 (K), D8.1 (K), D9.1 (K)
- net DN: now also R2.1
- net DP: now also R10.1
- net GND: now also C10.2, J3.A1B12 (GND), J3.B1A12 (GND), J3.S1 (SHIELD), J3.S2 (SHIELD), J3.S3 (SHIELD), J3.S4 (SHIELD), R1.2, R11.1
- new net: J3.A5 (CC1), R1.1
- new net: J3.A6 (DP1), J3.B6 (DP2), R10.2
- new net: J3.A7 (DN1), J3.B7 (DN2), R2.2
- new net: J3.B5 (CC2), R11.2
- new net Row_2: D13.1 (K), D18.1 (K), D22.1 (K), D26.1 (K), D3.1 (K), D30.1 (K), D35.1 (K), D39.1 (K), D43.1 (K), D47.1 (K), D52.1 (K), D57.1 (K), D64.1 (K), D8.1 (K)
- new net Row_3: D14.1 (K), D19.1 (K), D23.1 (K), D27.1 (K), D31.1 (K), D36.1 (K), D4.1 (K), D40.1 (K), D44.1 (K), D48.1 (K), D53.1 (K), D58.1 (K), D63.1 (K), D9.1 (K)
- no-connect marks 3 -> 2
Other:
- moved on the sheet: J1

Commit message: Layout almost finished 2.0
Parts:
- J1: footprint acheron_Connectors:PinHeader_1x6_P2.54mm_Vertical -> acheron_Connectors:PinHeader_2x3_P2.54mm_Vertical
Connections:
- net Col_0: now also U1.28 (PB4)
- net Col_1: now also U1.29 (PB5)
- net Col_10: now also U1.20 (PD2)
- net Col_11: now also U1.21 (PD3)
- net Col_12: now also U1.25 (PD4)
- net Col_13: now also U1.22 (PD5)
- net Col_2: now also U1.30 (PB6)
- net Col_3: now also U1.31 (PC6)
- net Col_4: now also U1.32 (PC7)
- net Col_5: now also U1.38 (PF5)
- net Col_6: now also U1.37 (PF6)
- net Col_7: now also U1.8 (PB0)
- net Col_8: now also U1.18 (PD0)
- net Col_9: now also U1.19 (PD1)
- net Row_0: now also U1.1 (PE6)
- net Row_1: now also U1.39 (PF4)
- net Row_2: now also U1.41 (PF0)
- net Row_3: now also U1.40 (PF1)
- net Row_4: now also U1.36 (PF7)
- no-connect marks 2 -> 5
Changed lines of the file:
@@
 F 0 "J1" H 7721 9096 50  0000 R CNN
 F 1 "AVR-ISP-6" H 7721 9005 50  0000 R CNN
-F 2 "acheron_Connectors:PinHeader_1x6_P2.54mm_Vertical" V 7800 9050 50  0001 C CNN
+F 2 "acheron_Connectors:PinHeader_2x3_P2.54mm_Vertical" V 7800 9050 50  0001 C CNN
 F 3 " ~" H 6775 8450 50  0001 C CNN
 	1    8050 9000
@@
 Connection ~ 15200 5400
 Connection ~ 15200 4250
+Text GLabel 3400 9750 2    50   Input ~ 0
+Row_0
+Text GLabel 3400 10450 2    50   Input ~ 0
+Row_4
+Text GLabel 3400 10150 2    50   Input ~ 0
+Row_1
+Text GLabel 3400 10050 2    50   Input ~ 0
+Row_3
+Text GLabel 3400 9950 2    50   Input ~ 0
+Row_2
+Text GLabel 3400 7950 2    50   Input ~ 0
+Col_0
+Text GLabel 3400 8050 2    50   Input ~ 0
+Col_1
+Text GLabel 3400 8150 2    50   Input ~ 0
+Col_2
+Text GLabel 3400 8450 2    50   Input ~ 0
+Col_3
+Text GLabel 3400 8550 2    50   Input ~ 0
+Col_4
+Text GLabel 3400 10350 2    50   Input ~ 0
+Col_6
+Text GLabel 3400 10250 2    50   Input ~ 0
+Col_5
+Text GLabel 3400 8750 2    50   Input ~ 0
+Col_8
+Text GLabel 3400 8850 2    50   Input ~ 0
+Col_9
+Text GLabel 3400 7550 2    50   Input ~ 0
+Col_7
+Text GLabel 3400 8950 2    50   Input ~ 0
+Col_10
+Text GLabel 3400 9050 2    50   Input ~ 0
+Col_11
+Text GLabel 3400 9150 2    50   Input ~ 0
+Col_12
+Text GLabel 3400 9250 2    50   Input ~ 0
+Col_13
+NoConn ~ 3400 9350
+NoConn ~ 3400 9450
+NoConn ~ 3400 8250
 $EndSCHEMATC

Commit message: Almost finished (no revision yet)
Parts:
- added D65: PRTR5V0U2X, Package_TO_SOT_SMD:SOT-143, symbol Power_Protection:PRTR5V0U2X
- added F1: 500mA, Fuse:Fuse_1210_3225Metric_Pad1.42x2.65mm_HandSolder, symbol Device:Fuse_Small
Connections:
- net +5V: now also F1.2; no longer J3.A4B9 (VBUS), J3.B4A9 (VBUS)
- net GND: now also D65.1 (GND)
- net XTAL1: now reaches C1.1, U1.17 (XTAL1), Y1.1
- net XTAL2: now reaches C2.1, U1.16 (XTAL2), Y1.2
- net at J3.A6 (DP1), J3.B6 (DP2), R10.2: now also D65.2 (I/O1)
- net at J3.A7 (DN1), J3.B7 (DN2), R2.2: now also D65.3 (I/O2)
- new net VCC: D65.4 (VCC), F1.1, J3.A4B9 (VBUS), J3.B4A9 (VBUS)
Other:
- moved on the sheet: C1, C10, C2, C3, C4, C5, C6, C7, C8, C9, J1, J3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

Commit message: GRAPHICS
Other:
- note added: "RESET\n"
- note added: "SWITCH MATRIX"
- note added: "USB TYPE-C\n"
- note removed: "RESET"
- note removed: "USB\n"
- moved on the sheet: C10, C4, C5, C7, C8, C9, D65, F1, J3, R1, R10, R11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
