File: A_Key_V1.1.kicad_pcb (KiCad board)
At the start: 2 copper layers, 290.5 x 100 mm, 151 parts, among them J1 AVR-ISP-6, J2 TYPE-C-31-M12_13, SW1 SW_Push, SW10 [>], SW11 [Win], SW12 [2], SW13 [W], SW14 [S], SW15 [Z], SW16 [Alt], SW17 [3], SW18 [E], SW19 [D], SW2 [\], SW20 [X], SW21 [4], SW22 [R], SW23 [F], SW24 [C], SW25 [5], SW26 [T], SW27 [G], SW28 [V], SW29 [6], SW3 [LTab], SW30 [Y], SW31 [H], SW32 [B], SW33 [Space], SW34 [7], SW35 [U], SW36 [J], SW37 [N], SW38 [8], SW39 [I], SW4 [LCaps], SW40 [K], SW41 [M], SW42 [9], SW43 [O], SW44 [L], SW45 [;], SW46 [0], SW47 [P], SW48 [Ñ], SW49 [:], SW5 [LShift], SW50 [AltGr], SW51 [?], SW52 [^], SW53 [¨], SW54 [_], SW55 [Win], SW56 [¿], SW57 [*], SW58 [Ç], SW59 [RShift], SW6 [LCtrl], SW60 [Menu], SW61 [Backspc], SW62 [Enter1.5], SW63 [Ctrl2], SW64 [Unass], SW65 [Unass1.25], SW7 [1], SW8 [Q], SW9 [A], U1 ATmega32U4-AU, Y1 Crystal

Commit message: PCB Layout almost finished
Parts:
- removed the D1 at (47.8, 22.1)
- removed J2: TYPE-C-31-M12_13, TYPE-C-31-M-12:HRO_TYPE-C-31-M-12
- removed R6, R7: 5k, Resistor_SMD:R_0805_2012Metric_Pad1.20x1.40mm_HandSolder
- removed R8, R9: 22k, Resistor_SMD:R_0805_2012Metric_Pad1.20x1.40mm_HandSolder
- removed the SW2 at (79.8, 30.5)
- added C10: 100n, Capacitor_SMD:C_0805_2012Metric_Pad1.18x1.45mm_HandSolder, B.Cu at (153.4, -23.1)
- added J3: TYPE-C-31-M-12, TYPE-C-31-M-12:HRO_TYPE-C-31-M-12, B.Cu at (142.5, -111.3)
- added R1: 5k, Resistor_SMD:R_0805_2012Metric_Pad1.20x1.40mm_HandSolder, B.Cu at (135.9, -111.5)
- added R10: 22k, Resistor_SMD:R_0805_2012Metric_Pad1.20x1.40mm_HandSolder, B.Cu at (143.8, -102.6)
- added R11: 5k, Resistor_SMD:R_0805_2012Metric_Pad1.20x1.40mm_HandSolder, B.Cu at (149.1, -111.5)
- added R2: 22k, Resistor_SMD:R_0805_2012Metric_Pad1.20x1.40mm_HandSolder, B.Cu at (141.7, -102.6)
- C4: value 0.1u -> 10u
- C5: value 0.1u -> 1u
- C7, C8: value 0.1u -> 100n
- C9: value 10u -> 1u
- D63, D64, SW59, SW62, SW64, SW65: moved to B.Cu
- moved D3 302.9 mm to (17.9, -63.1), turned to 90 degrees
- moved D16 295.6 mm to (67.9, -101.2), turned to 90 degrees
- moved D11 279.8 mm to (48.9, -101.2), turned to 90 degrees
- moved D24 267.4 mm to (106.0, -101.2), turned to 90 degrees
- moved D7 265.1 mm to (39.4, -82.2), turned to 90 degrees
- moved D12 261.3 mm to (58.4, -82.2), turned to 90 degrees
- moved D13 245.4 mm to (63.2, -63.1), turned to 90 degrees
- moved D18 238.6 mm to (82.2, -63.1), turned to 90 degrees
- moved D19 230.6 mm to (72.7, -44.1), turned to 90 degrees
- moved D6 226.8 mm to (29.8, -101.2), turned to 90 degrees
- moved D4 226.6 mm to (13.2, -44.1), turned to 90 degrees
- moved D8 221.4 mm to (44.1, -63.1), turned to 90 degrees
- moved D30 219.3 mm to (143.0, -59.5), turned to 0 degrees
- moved D27 216.5 mm to (110.8, -44.1), turned to 90 degrees
- moved D31 211.7 mm to (129.9, -44.1), turned to 90 degrees
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Connections:
- D13 pad 1: Col_13 -> Row_2
- D14 pad 1: Col_13 -> Row_3
- D18 pad 1: Col_13 -> Row_2
- D19 pad 1: Col_13 -> Row_3
- D22 pad 1: Col_13 -> Row_2
- D23 pad 1: Col_13 -> Row_3
- D26 pad 1: Col_13 -> Row_2
- D27 pad 1: Col_13 -> Row_3
- D3 pad 1: Col_13 -> Row_2
- D30 pad 1: Col_13 -> Row_2
- D31 pad 1: Col_13 -> Row_3
- D35 pad 1: Col_13 -> Row_2
- D36 pad 1: Col_13 -> Row_3
- D39 pad 1: Col_13 -> Row_2
- D4 pad 1: Col_13 -> Row_3
- D40 pad 1: Col_13 -> Row_3
- D43 pad 1: Col_13 -> Row_2
- D44 pad 1: Col_13 -> Row_3
- D47 pad 1: Col_13 -> Row_2
- D48 pad 1: Col_13 -> Row_3
- D52 pad 1: Col_13 -> Row_2
- D53 pad 1: Col_13 -> Row_3
- D57 pad 1: Col_13 -> Row_2
- D58 pad 1: Col_13 -> Row_3
- D63 pad 1: Col_13 -> Row_3
- D64 pad 1: Col_13 -> Row_2
- D8 pad 1: Col_13 -> Row_2
- D9 pad 1: Col_13 -> Row_3
- SW65 pad 1: Net-(SW65-Pad1) -> Col_13
- U1 pad 42: Net-(U1-Pad42) -> +5V
Routing:
- net Row_3: track 0.00 -> 279.7 mm, vias 0 -> 4
- net Row_1: track 0.00 -> 279.6 mm, vias 0 -> 4
- net Row_4: track 0.00 -> 269.9 mm
- net Row_2: track 0.00 -> 269.9 mm, vias 0 -> 4
- net Row_0: track 0.00 -> 236.2 mm, vias 0 -> 4
- net GND: track 0.02 -> 229.2 mm
- net +5V: track 0.00 -> 195.8 mm, vias 0 -> 9
- net Col_10: track 0.00 -> 104.1 mm
- net Col_11: track 0.00 -> 103.2 mm
- net Col_12: track 0.00 -> 101.6 mm
- net Col_1: track 0.00 -> 100.5 mm
- net Col_0: track 0.00 -> 97.0 mm
- net Col_2: track 0.00 -> 96.0 mm
- net Col_13: track 0.00 -> 93.3 mm
- net Col_5: track 0.00 -> 93.1 mm
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
Commit message: Layout almost finished 2.0
Parts:
- added K_CTRL1: MX-1.25U, MX_Alps_Hybrid:MX-1.25U, F.Cu at (21.4, -26.1)
- added K_CTRL1: MX-1.25U, MX_Alps_Hybrid:MX-1.25U, F.Cu at (28.0, 81.4)
- added K_CTRL2: MX-1.5U, MX_Alps_Hybrid:MX-1.5U-FLIPPED, F.Cu at (23.8, -26.1)
- added K_CTRL2: MX-1.5U, MX_Alps_Hybrid:MX-1.5U-FLIPPED, F.Cu at (30.4, 81.4)
- added REF**: 60_Outline, locallib:60_Outline-Modded, F.Cu at (152.4, -64.2)
- added REF**: 60_Outline, locallib:60_Outline-Modded, F.Cu at (159.0, 43.3)
- J1: footprint acheron_Connectors:PinHeader_1x6_P2.54mm_Vertical -> acheron_Connectors:PinHeader_2x3_P2.54mm_Vertical
- SW33: moved to B.Cu
- moved R5 13.7 mm to (197.4, -34.3)
- moved C7 4.56 mm to (168.0, -35.1), turned to 180 degrees
- moved R1 3.93 mm to (132.7, -109.3)
- moved C5 3.33 mm to (165.6, -38.6)
- moved R3 2.66 mm to (153.2, -20.1)
- moved R11 2.63 mm to (150.4, -109.3)
- moved J3 2.38 mm to (142.4, -113.6)
- moved C9 2.21 mm to (154.0, -31.5)
- moved C4 1.79 mm to (169.2, -18.1)
- moved C2 1.49 mm to (172.7, -27.2)
- moved J1 1.02 mm to (185.8, -27.0)
- moved C8 1.00 mm to (157.6, -35.3), turned to 90 degrees
- moved C10 1.00 mm to (153.2, -22.1), turned to 180 degrees
- moved C1 0.98 mm to (172.7, -23.4)
- moved Y1 0.78 mm to (175.8, -25.4)
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Connections:
- U1 pad 1: Net-(U1-Pad1) -> Row_0
- U1 pad 18: Net-(U1-Pad18) -> Col_8
- U1 pad 19: Net-(U1-Pad19) -> Col_9
- U1 pad 20: Net-(U1-Pad20) -> Col_10
- U1 pad 21: Net-(U1-Pad21) -> Col_11
- U1 pad 22: Net-(U1-Pad22) -> Col_13
- U1 pad 25: Net-(U1-Pad25) -> Col_12
- U1 pad 28: Net-(U1-Pad28) -> Col_0
- U1 pad 29: Net-(U1-Pad29) -> Col_1
- U1 pad 30: Net-(U1-Pad30) -> Col_2
- U1 pad 31: Net-(U1-Pad31) -> Col_3
- U1 pad 32: Net-(U1-Pad32) -> Col_4
- U1 pad 36: Net-(U1-Pad36) -> Row_4
- U1 pad 37: Net-(U1-Pad37) -> Col_6
- U1 pad 38: Net-(U1-Pad38) -> Col_5
- U1 pad 39: Net-(U1-Pad39) -> Row_1
- U1 pad 40: Net-(U1-Pad40) -> Row_3
- U1 pad 41: Net-(U1-Pad41) -> Row_2
- U1 pad 8: Net-(U1-Pad8) -> Col_7
Routing:
- net Col_0: track 97.0 -> 243.8 mm
- net Col_13: track 93.3 -> 225.2 mm, vias 0 -> 2
- net Col_1: track 100.5 -> 221.8 mm
- net Col_12: track 101.6 -> 217.3 mm, vias 0 -> 1
- net Col_3: track 74.5 -> 178.4 mm, vias 0 -> 1
- net Col_2: track 96.0 -> 192.9 mm, vias 0 -> 2
- net Col_11: track 103.2 -> 188.0 mm, vias 0 -> 1
- net Col_4: track 71.8 -> 152.8 mm, vias 0 -> 1
- net Row_0: track 236.2 -> 312.9 mm
- net Row_1: track 279.6 -> 342.0 mm, vias 4 -> 6
- net Col_10: track 104.1 -> 163.7 mm, vias 0 -> 1
- net +5V: track 195.8 -> 254.5 mm, vias 9 -> 15
- net Col_5: track 93.1 -> 141.6 mm, vias 0 -> 1
- net /RST: track 15.6 -> 62.6 mm
- net Col_9: track 78.0 -> 124.1 mm, vias 0 -> 1
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- added copper zone on B.Cu, net GND
Other:
- board size 290.5 x 100 mm -> 285 x 98.1 mm

Commit message: Almost finished (no revision yet)
Parts:
- removed K_CTRL1 (x2): MX-1.25U, MX_Alps_Hybrid:MX-1.25U
- removed K_CTRL2 (x2): MX-1.5U, MX_Alps_Hybrid:MX-1.5U-FLIPPED
- removed the REF** at (159.0, 43.3)
- added D65: PRTR5V0U2X, Package_TO_SOT_SMD:SOT-143, B.Cu at (142.6, -102.5)
- added F1: 500mA, Fuse:Fuse_1210_3225Metric_Pad1.42x2.65mm_HandSolder, B.Cu at (146.6, -97.3)
- moved R2 11.8 mm to (136.3, -92.1)
- moved R10 11.8 mm to (138.4, -92.1)
- moved SW1 11.0 mm to (203.0, -35.1), turned to 90 degrees
- moved D49 10.7 mm to (209.4, -34.1), turned to 180 degrees
- moved J1 6.71 mm to (183.0, -33.1)
- moved C2 4.10 mm to (176.8, -27.3), turned to 270 degrees
- moved C1 4.07 mm to (176.8, -23.4), turned to 90 degrees
- moved C6 3.70 mm to (195.9, -34.8)
- moved R4 3.68 mm to (198.2, -34.8)
- moved R5 3.57 mm to (197.2, -37.9)
- moved D7 3.40 mm to (39.7, -78.8)
- moved D61 2.68 mm to (265.0, -79.5)
- moved C4 2.34 mm to (167.7, -19.8), turned to 90 degrees
- moved Y1 2.22 mm to (173.7, -26.1)
- moved R3 1.63 mm to (153.8, -21.6), turned to 270 degrees
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Connections:
- net Net-(C1-Pad1) renamed /XTAL1
- net Net-(C2-Pad1) renamed /XTAL2
- J3 pad A4B9: +5V -> VCC
- J3 pad B4A9: +5V -> VCC
Routing:
- net +5V: track 254.5 -> 222.9 mm, vias 15 -> 14
- net VCC: track 0.00 -> 26.5 mm, vias 0 -> 4
- net Net-(D65-Pad3): track 7.50 -> 23.7 mm
- net Net-(D65-Pad2): track 9.03 -> 24.5 mm
- net GND: track 234.6 -> 248.2 mm, vias 18 -> 20
- net Row_0: track 312.9 -> 324.7 mm
- net Row_1: track 342.0 -> 351.7 mm
- net /DP: track 86.0 -> 78.9 mm
- net /DN: track 86.0 -> 78.9 mm
- net Net-(D61-Pad2): track 12.4 -> 18.2 mm
- net Row_4: track 298.7 -> 304.2 mm, vias 3 -> 4
- net /MISO: track 22.3 -> 16.9 mm
- net /SCK: track 24.4 -> 19.1 mm
- net /MOSI: track 26.7 -> 21.5 mm
- net Row_2: track 309.7 -> 304.8 mm, vias 6 -> 7
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Other:
- rule trace_min: 0.2 -> 0.1
- board text added: "PCB Revision 1.0"
- board text added: "RatBoard"

Commit message: Almost finished
Other:
- board text added: "RATBOARD"
- board text added: "RatBoard v1.0 Ana Povea"
- board text added: "v1.0 APR"

Commit message: GRAPHICS
Other:
- board size 285 x 98.1 mm -> 285 x 101.6 mm
- board text removed: "RatBoard"

Commit message: final
Routing:
- net GND: track 248.2 -> 252.2 mm, vias 20 -> 21
- net Net-(D65-Pad3): track 23.7 -> 25.9 mm, vias 0 -> 1
- net /DP: track 78.9 -> 77.5 mm
- net /DN: track 78.9 -> 77.6 mm
- net Net-(D65-Pad2): track 24.5 -> 25.3 mm, vias 0 -> 1
- net +5V: track 222.9 -> 223.7 mm
- net VCC: track 26.5 -> 25.9 mm
Other:
- net class +5V added: clearance 0.2, trace_width 0.4, via_dia 0.8, via_drill 0.4
- rule trace_min: 0.1 -> 0.2
